Commit message: Rebase from 'upstream'

File: abb_resources/urdf/common_colours.xacro (robot description, xacro)
@@ -27,4 +27,6 @@
   <!-- RAL 6002 leaf green -->
   <xacro:property name="colour_abb_leaf_green" value="0.1764706 0.3529412 0.1529412 1" />
+  <!-- RAL 6003 olive green -->
+  <xacro:property name="colour_abb_olive_green" value="${ 80/255} ${ 83/255} ${ 60/255} 1" />
   <!-- RAL 9002 gray white -->
   <xacro:property name="colour_abb_gray_white" value="0.8392157 0.8352941 0.7921569 1" />

File: abb_resources/urdf/common_materials.xacro (robot description, xacro)
@@ -57,4 +57,9 @@
     </material>
   </xacro:macro>
+  <xacro:macro name="material_abb_olive_green">
+    <material name="">
+      <color rgba="${colour_abb_olive_green}"/>
+    </material>
+  </xacro:macro>
   <xacro:macro name="material_abb_gray_white">
     <material name="">
